Commit message: upload

File: urdf/robot2.xacro (robot description, xacro)
@@ -74,17 +74,4 @@
       </geometry>
     </visual>
-  <!-- caster rear
-  <collision name="caster_rear_collision">
-    <origin rpy=" 0 0 0" xyz="-0.35 0 -0.05"/>
-    <geometry>
-      <sphere radius="0.05"/>
-    </geometry>
-  </collision>
-  <visual name="caster_rear_visual">
-    <origin rpy=" 0 0 0" xyz="-0.2 0 -0.05"/>
-    <geometry>
-      <sphere radius="0.05"/>
-    </geometry>
-  </visual> -->
 </link>
   <link name="link_right_wheel">
